File: sram-cell.sch (KiCad schematic (older format))
At the start: 59 parts, among them J1 USB_B_Micro, J2 PowerHeader, Q1 PMOS_GSD, Q10 NMOS_GSD, Q11 NMOS_GSD, Q2 PMOS_GSD, Q3 NMOS_GSD, Q4 NMOS_GSD, Q5 NMOS_GSD, Q6 NMOS_GSD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

Commit message: final v1 boards
Parts:
- SW1: Link (none) -> https://www.mouser.com/ProductDetail/FSM4JAH
Changed lines of the file:
@@
 F 2 "Button_Switch_THT:SW_PUSH_6mm" H 2550 1800 50  0001 C CNN
 F 3 "~" H 2550 1800 50  0001 C CNN
+F 4 "https://www.mouser.com/ProductDetail/FSM4JAH" H 2550 1600 50  0001 C CNN "Link"
 	1    2550 1600
 	1    0    0    -1
